File: optoCouplerDmb.sch (EAGLE design)
At the start: 19 parts, among them U1 6N137, U2 6N137

Commit message: resistors 10mm , added led
Parts:
- added LED3: (no value), led:LED3MM
- added R5: 1k, rcl:R-EU_0207/10
- R1, R2, R3, R4: device rcl:R-EU_0204/7 -> rcl:R-EU_0207/10
Connections:
- new net N$3: LED3.C, R5.2
- net GND: now also R5.1
- net VCC: now also LED3.A
Other:
- moved on the sheet: C1, D1, D2, F1, H1, H2, H3, H4, LED1, LED2, R1, R2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
